Commit message: adding link visuals

File: urdf/learm.urdf (robot description, URDF)
Before this commit: robot LeArm, 8 links, 7 joints
Links:
- link base_link: geometry visual cylinder length=0.070 radius=0.060
- link forearm_link: geometry visual box size=0.025 0.055 0.110
- link grip_left_link: geometry visual box size=0.010 0.012 0.096
- link grip_right_link: geometry visual box size=0.010 0.012 0.096
- link hand_link: geometry visual box size=0.055 0.057 0.052
- link humerus_link: geometry visual box size=0.025 0.055 0.130
- link shoulder_link: geometry visual cylinder length=0.012 radius=0.040
- link wrist_link: geometry visual box size=0.058 0.045 0.070
Joints:
- joint elbow: origin xyz=0 0 0.105 rpy=0 0 0 -> xyz=0 0 0.105
- joint grip_left: origin xyz=0 +0.015 0.035 rpy=0 0 0 -> xyz=0 +0.015 0.035
- joint grip_right: origin xyz=0 -0.015 0.035 rpy=0 0 0 -> xyz=0 -0.015 0.035
- joint shoulder_lift: origin xyz=0 0 0.015 rpy=0 0 0 -> xyz=0 0 0.015
- joint shoulder_pan: origin xyz=0 0 0.070 rpy=0 0 0 -> xyz=0 0 0.070
- joint wrist_flex: origin xyz=0 0 0.090 rpy=0 0 0 -> xyz=0 0 0.090
- joint wrist_roll: origin xyz=0 0 0.065 rpy=0 0 0 -> xyz=0 0 0.065

Commit message: starting to add models from manufacturer

File: urdf/learm.urdf (robot description, URDF)
Before this commit: robot LeArm, 8 links, 7 joints
Links:
- link base_link: geometry visual mesh filename=package://learm-ros/meshes/base.stl scale=0.001 0.001 0.001
- link shoulder_link: geometry visual mesh filename=package://learm-ros/meshes/shoulder.stl scale=0.001 0.001 0.001
Joints:
- joint shoulder_pan: origin xyz=0 0 0.070 -> xyz=0 0 0.059

Commit message: adding humerus

File: urdf/learm.urdf (robot description, URDF)
Before this commit: robot LeArm, 8 links, 7 joints
Links:
- link humerus_link: geometry visual mesh filename=package://learm-ros/meshes/humerus.stl scale=0.001 0.001 0.001
Joints:
- joint shoulder_lift: origin xyz=0 0 0.015 -> xyz=-0.010 0 0.028

Commit message: adding forearm

File: urdf/learm.urdf (robot description, URDF)
Before this commit: robot LeArm, 8 links, 7 joints
Links:
- link forearm_link: geometry visual mesh filename=package://learm-ros/meshes/forearm.stl scale=0.001 0.001 0.001

Commit message: adding wrist

File: urdf/learm.urdf (robot description, URDF)
Before this commit: robot LeArm, 8 links, 7 joints
Links:
- link wrist_link: geometry visual mesh filename=package://learm-ros/meshes/wrist.stl scale=0.001 0.001 0.001

Commit message: adding hand

File: urdf/learm.urdf (robot description, URDF)
Before this commit: robot LeArm, 8 links, 7 joints
Links:
- link hand_link: geometry visual mesh filename=package://learm-ros/meshes/hand.stl scale=0.001 0.001 0.001

Commit message: use <mimic> to represent gripper kinematics

File: urdf/learm.urdf (robot description, URDF)
Before this commit: robot LeArm, 8 links, 7 joints
Links:
- added link finger_left_link; visual box size=0.010 0.012 0.096
- added link finger_right_link; visual box size=0.010 0.012 0.096
- added link tendon_left_link; visual box size=0.010 0.012 0.096
- added link tendon_right_link; visual box size=0.010 0.012 0.096
Joints:
- added joint finger_left: type revolute, parent grip_left_link, child finger_left_link, origin xyz=0 0 0.031, axis 1 0 0, limit lower=-1.57 upper=0 effort=1000 velocity=0.5, mimic joint=grip_left multiplier=-1
- added joint finger_right: type revolute, parent grip_right_link, child finger_right_link, origin xyz=0 0 0.031, axis 1 0 0, limit lower=0 upper=1.57 effort=1000 velocity=0.5, mimic joint=grip_left
- added joint tendon_left: type revolute, parent hand_link, child tendon_left_link, origin xyz=0 +0.005 0.050, axis 1 0 0, limit lower=-1.57 upper=0 effort=1000 velocity=0.5, mimic joint=grip_left
- added joint tendon_right: type revolute, parent hand_link, child tendon_right_link, origin xyz=0 -0.005 0.050, axis 1 0 0, limit lower=0 upper=1.57 effort=1000 velocity=0.5, mimic joint=grip_left multiplier=-1
- joint grip_right: mimic (none) -> joint=grip_left multiplier=-1

Commit message: adding fingers

File: urdf/learm.urdf (robot description, URDF)
Before this commit: robot LeArm, 12 links, 11 joints
Links:
- link finger_left_link: geometry visual mesh filename=package://learm-ros/meshes/finger.stl scale=0.001 0.001 0.001
- link finger_right_link: geometry visual mesh filename=package://learm-ros/meshes/finger.stl scale=0.001 0.001 0.001

Commit message: scaling meshes by 0.001 in FreeCad (Mesh Design mode)

File: urdf/learm.urdf (robot description, URDF)
Before this commit: robot LeArm, 12 links, 11 joints
Links:
- link base_link: geometry visual mesh filename=package://learm-ros/meshes/base.stl
- link finger_left_link: geometry visual mesh filename=package://learm-ros/meshes/finger.stl
- link finger_right_link: geometry visual mesh filename=package://learm-ros/meshes/finger.stl
- link forearm_link: geometry visual mesh filename=package://learm-ros/meshes/forearm.stl
- link hand_link: geometry visual mesh filename=package://learm-ros/meshes/hand.stl
- link humerus_link: geometry visual mesh filename=package://learm-ros/meshes/humerus.stl
- link shoulder_link: geometry visual mesh filename=package://learm-ros/meshes/shoulder.stl
- link wrist_link: geometry visual mesh filename=package://learm-ros/meshes/wrist.stl

Commit message: Adding tendons

File: urdf/learm.urdf (robot description, URDF)
Before this commit: robot LeArm, 12 links, 11 joints
Links:
- link tendon_left_link: geometry visual mesh filename=package://learm-ros/meshes/tendon.stl
- link tendon_right_link: geometry visual mesh filename=package://learm-ros/meshes/tendon.stl

Commit message: left carpal

File: urdf/learm.urdf (robot description, URDF)
Before this commit: robot LeArm, 12 links, 11 joints
Links:
- link grip_left_link: geometry visual mesh filename=package://learm-ros/meshes/carpal-left.stl

Commit message: Adding Carpal-Right and first set of model corrections

File: urdf/learm.urdf (robot description, URDF)
Before this commit: robot LeArm, 12 links, 11 joints
Links:
- link grip_right_link: geometry visual mesh filename=package://learm-ros/meshes/carpal-right.stl
Joints:
- joint finger_left: origin xyz=0 0 0.031 -> xyz=0 0 0.030
- joint finger_right: origin xyz=0 0 0.031 -> xyz=0 0 0.030
- joint grip_left: origin xyz=0 +0.015 0.035 -> xyz=0 +0.015 0.030
- joint grip_right: origin xyz=0 -0.015 0.035 -> xyz=0 -0.015 0.030
- joint wrist_roll: origin xyz=0 0 0.065 -> xyz=0 0 0.060

Commit message: flipping shoulder_lift to match IRL robot

File: urdf/learm.urdf (robot description, URDF)
Before this commit: robot LeArm, 12 links, 11 joints
Joints:
- joint shoulder_lift: axis 0 1 0 -> 0 -1 0
